File: hardware/SolarDataLogger/SolarDataLogger.kicad_pcb (KiCad board)
At the start: 2 copper layers, 90 x 90 mm, 69 parts, among them CN1 WJ2EDGVC-5.08-2P, Q1 LBC847BDW1T1G, SW1 TS-1088-AR02016, SW2 TS-1088-AR02016, U1 AMS1117-3.3_C347222, U10 RH-5000, U11 RH-5000, U12 RH-5000, U13 CP2102N-A02-GQFN24R, U2 RH-5000, U3 TPS5430DDAR, U4 RH-5000, U5 RH-5000, U6 AHT20_C2757850, U7 HY2541WV-N-2X3P, U8 ESP32-C6-WROOM-1-N8, U9 RH-5000

Commit message: What?
Parts:
- removed CN1: WJ2EDGVC-5.08-2P, C8445-Greenplug:CONN-TH_WJ2EDGVC-5.08-2P
- added J1: 2305908-2, 2305908-2:23059082, F.Cu at (57.1, 73.7)
- added J2: 2213932-3, 2213932-3:22139323, F.Cu at (135.4, 73.4)
- moved D1 186.4 mm to (48.6, 160.1)
- moved L1 186.4 mm to (56.2, 154.2)
- moved U3 186.4 mm to (48.8, 154.9)
- moved D7 175.0 mm to (72.3, 31.8)
- moved C1 172.9 mm to (31.7, 168.0)
- moved C2 172.9 mm to (31.7, 170.6)
- moved C3 172.9 mm to (31.7, 173.1)
- moved C4 172.9 mm to (31.7, 175.6)
- moved C6 172.9 mm to (31.7, 178.1)
- moved C8 172.9 mm to (31.7, 183.1)
- moved C9 172.9 mm to (31.7, 185.6)
- moved R6 172.9 mm to (39.8, 170.6)
- moved R7 172.9 mm to (39.8, 173.1)
- moved R1 172.9 mm to (35.8, 178.1)
- moved R2 172.9 mm to (35.8, 180.6)
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Other:
- outline, holes or cut-outs redrawn
- copper layers 2 -> 6

Commit message: The work must be done
Parts:
- moved C9 135.1 mm to (114.0, 78.5), turned to 90 degrees
- moved R7 119.2 mm to (112.3, 78.5), turned to -90 degrees
- moved R3 109.8 mm to (84.1, 76.5)
- moved C8 109.1 mm to (114.0, 111.4), turned to -90 degrees
- moved D11 105.5 mm to (77.5, 78.5), turned to -90 degrees
- moved R4 104.1 mm to (88.1, 74.0), turned to 90 degrees
- moved R14 102.7 mm to (76.7, 81.0)
- moved D12 102.4 mm to (79.5, 78.5), turned to -90 degrees
- moved C7 101.7 mm to (87.0, 69.7)
- moved Q1 101.5 mm to (85.7, 74.1), turned to 90 degrees
- moved R15 98.3 mm to (80.3, 81.0), turned to 180 degrees
- moved R16 98.2 mm to (74.9, 72.6)
- moved R17 97.9 mm to (74.9, 74.4)
- moved R6 96.3 mm to (115.8, 111.4), turned to 90 degrees
- moved D2 95.6 mm to (109.6, 87.1), turned to 180 degrees
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Connections:
- C8 pad 2: Net-(C8-Pad2) -> /GPIO9
- C9 pad 2: Net-(C9-Pad2) -> /CHIP_PU
- D8 pad 2: unconnected-(D8-Pad2) -> /D-
- J1 pad 1: GND -> Net-(U3-VIN)
- J1 pad 2: Net-(U3-VIN) -> GND
- J2 pad 3: /V_GND -> GND
- R6 pad 1: Net-(C8-Pad2) -> /GPIO9
- R7 pad 1: Net-(C9-Pad2) -> /CHIP_PU
Routing:
- added copper zone on In1.Cu, net GND
- added copper zone on In4.Cu, net GND

Commit message: Templates for all!
Parts:
- U7: footprint C17179450-2x3-IDC-Header:HDR-TH_6P-P2.54-V-F-R2-C3-S2.54-4 -> Connector_IDC:IDC-Header_2x03_P2.54mm_Vertical_SMD
- moved H5 3.61 mm to (95.0, 82.0)
- moved H6 3.00 mm to (95.0, 108.0)
- turned U7 to -90 degrees
