File: hardware/SolarDataLogger/SolarDataLogger.kicad_sch (KiCad schematic)
At the start: 67 parts, among them CN1 WJ2EDGVC-5.08-2P, Q1 LBC847BDW1T1G, SW1 TS-1088-AR02016, SW2 TS-1088-AR02016, U1 AMS1117-3.3_C347222, U10 RH-5000, U11 RH-5000, U12 RH-5000, U13 CP2102N-A02-GQFN24R, U2 RH-5000, U3 TPS5430DDAR, U4 RH-5000, U5 RH-5000, U6 AHT20_C2757850, U7 HY2541WV-N-2X3P, U8 ESP32-C6-WROOM-1-N8, U9 RH-5000

Commit message: Moving along
Parts:
- added H6: MountingHole_Pad, MountingHole:MountingHole_3.5mm_Pad_TopBottom, symbol Mechanical:MountingHole_Pad
- added R17: 1k, Resistor_SMD:R_0603_1608Metric, symbol Device:R_Small_US
- C1, C10, C11, C12, C13, C2, C3, C4, C6, C7, C8, C9: footprint (none) -> Capacitor_SMD:C_0603_1608Metric
- C5: footprint (none) -> C125977-220uF-Cap:CAP-SMD_BD10.0-L10.3-W10.3-LS11.3-FD
- D11, D12: footprint (none) -> LED_SMD:LED_0603_1608Metric
- H1, H2, H3, H4, H5: footprint (none) -> MountingHole:MountingHole_3.5mm_Pad_TopBottom
- R1, R10, R11, R12, R13, R14, R15, R16, R2, R3, R4, R5, R6, R7, R8, R9: footprint (none) -> Resistor_SMD:R_0603_1608Metric
- U8: footprint ESP32-C6-WROOM-1-N8:XCVR_ESP32-C6-WROOM-1-N8 -> ESP32-C6-WROOM-1:XCVR_ESP32-C6-WROOM-1-N8
Connections:
- net D-: no longer D8.2
- net GND: now also H6.1
- net VCC: now also U13.5 (VIO), R17.1
- net at U13.9 (RSTb): now also R17.2
- no-connect marks 33 -> 32
Other:
- note added: "USB UART BRIDGE"
- company: (none) -> Eric Dynowski
- title: (none) -> Solar Data Logger
- moved on the sheet: C1, C10, C11, C12, C13, C2, C3, C4, C5, C6, C7, C8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

Commit message: What?
Parts:
- removed CN1: WJ2EDGVC-5.08-2P, C8445-Greenplug:CONN-TH_WJ2EDGVC-5.08-2P, symbol C8445-Greenplug:WJ2EDGVC-5.08-2P
- added J1: 2305908-2, 23059082, symbol 2305908-2:2305908-2
- added J2: 2213932-3, 22139323, symbol 2213932-3:2213932-3
Connections:
- net GND: now also J1.1
- net V_RXD: now also J2.1
- net V_TXD: now also J2.2
- net at C2.2, C3.2, U3.7 (VIN): now also J1.2
- new net V_GND: J2.3
Other:
- note added: "VICTRON CONNECTOR"
- moved on the sheet: C10, D3, D4, D5, D6, R8, R9, USB1

Commit message: The work must be done
Connections:
- net V_GND is gone; now on net GND: J2.3
- net CHIP_PU: now also C9.2, R7.1
- net D-: now also D8.2
- net GND: now also J1.2; no longer J1.1
- net GPIO9: now also C8.2, R6.1
- net at C2.2, C3.2, U3.7 (VIN): now also J1.1; no longer J1.2
- no-connect marks 32 -> 31
Other:
- moved on the sheet: J1

Commit message: Templates for all!
Parts:
- J1: footprint 23059082 -> 2305908-2:23059082
- J2: footprint 22139323 -> 2213932-3:22139323
- U7: footprint C17179450-2x3-IDC-Header:HDR-TH_6P-P2.54-V-F-R2-C3-S2.54-4 -> Connector_IDC:IDC-Header_2x03_P2.54mm_Vertical_SMD
Changed lines of the file:
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@@
 	(label "SCL"
 		(at 269.24 156.21 0)
+		(fields_autoplaced yes)
 		(effects
 			(font
@@
 	(label "GPIO9"
 		(at 67.31 265.43 0)
+		(fields_autoplaced yes)
 		(effects
 			(font
@@
 	(label "SDA"
 		(at 246.38 71.12 0)
+		(fields_autoplaced yes)
 		(effects
 			(font
@@
 	(label "TXD0"
 		(at 265.43 153.67 0)
+		(fields_autoplaced yes)
 		(effects
 			(font
@@
 	(label "USB_D+"
 		(at 265.43 146.05 0)
+		(fields_autoplaced yes)
 		(effects
 			(font
@@
 	(label "CHIP_PU"
 		(at 314.96 48.26 0)
+		(fields_autoplaced yes)
 		(effects
 			(font
@@
 	(label "GPIO8"
 		(at 364.49 99.06 0)
+		(fields_autoplaced yes)
 		(effects
 			(font
@@
 	(label "V_TXD"
 		(at 322.58 142.24 0)
+		(fields_autoplaced yes)
 		(effects
 			(font
@@
 	(label "V_TXD"
 		(at 265.43 140.97 0)
+		(fields_autoplaced yes)
 		(effects
 			(font
@@
 	(label "SCL"
 		(at 264.16 71.12 0)
+		(fields_autoplaced yes)
 		(effects
 			(font
@@
 	(label "TXD0"
 		(at 238.76 121.92 0)
+		(fields_autoplaced yes)
 		(effects
 			(font
@@
 	(label "RXD0"
 		(at 265.43 151.13 0)
+		(fields_autoplaced yes)
 		(effects
 			(font
@@
 	(label "RXD0"
 		(at 261.62 121.92 0)
+		(fields_autoplaced yes)
 		(effects
 			(font
@@
 	(label "TXD0"
 		(at 195.58 63.5 0)
+		(fields_autoplaced yes)
 		(effects
 			(font
@@
 	(label "SDA"
 		(at 270.51 43.18 0)
+		(fields_autoplaced yes)
 		(effects
 			(font
@@
 	(label "GPIO8"
 		(at 215.9 163.83 0)
+		(fields_autoplaced yes)
 		(effects
 			(font
@@
 	(label "D+"
 		(at 135.89 66.04 0)
+		(fields_autoplaced yes)
 		(effects
 			(font
@@
 	(label "RXD0"
 		(at 195.58 60.96 0)
+		(fields_autoplaced yes)
 		(effects
 			(font
@@
 	(label "SCL"
 		(at 240.03 43.18 0)
+		(fields_autoplaced yes)
 		(effects
 			(font
@@
 	(label "GPIO2"
 		(at 264.16 73.66 0)
+		(fields_autoplaced yes)
 		(effects
 			(font
@@
 	(label "D-"
 		(at 135.89 63.5 0)
+		(fields_autoplaced yes)
 		(effects
 			(font
@@
 	(label "D-"
 		(at 88.9 63.5 0)
+		(fields_autoplaced yes)
 		(effects
 			(font
@@
 	(label "GPIO1"
 		(at 214.63 146.05 0)
+		(fields_autoplaced yes)
 		(effects
 			(font
@@
 	(label "USB_D-"
 		(at 91.44 140.97 0)
+		(fields_autoplaced yes)
 		(effects
 			(font
@@
 	(label "USB_D-"
 		(at 265.43 143.51 0)
+		(fields_autoplaced yes)
 		(effects
 			(font
@@
 	(label "RTS"
 		(at 195.58 58.42 0)
+		(fields_autoplaced yes)
 		(effects
 			(font
@@
 	(label "GPIO9"
 		(at 215.9 166.37 0)
+		(fields_autoplaced yes)
 		(effects
 			(font
@@
 	(label "RTS"
 		(at 355.6 48.26 0)
+		(fields_autoplaced yes)
 		(effects
 			(font
@@
 	(label "USB_D+"
 		(at 91.44 138.43 0)
+		(fields_autoplaced yes)
 		(effects
 			(font
@@
 	(label "CHIP_PU"
 		(at 214.63 138.43 0)
+		(fields_autoplaced yes)
 		(effects
 			(font
@@
 	(label "V_RXD"
 		(at 265.43 138.43 0)
+		(fields_autoplaced yes)
 		(effects
 			(font
@@
 	(label "DTR"
 		(at 314.96 43.18 0)
+		(fields_autoplaced yes)
 		(effects
 			(font
@@
 	(label "D+"
 		(at 88.9 66.04 0)
+		(fields_autoplaced yes)
 		(effects
 			(font
@@
 	(label "GPIO2"
 		(at 214.63 148.59 0)
+		(fields_autoplaced yes)
 		(effects
 			(font
@@
 	(label "SDA"
 		(at 269.24 158.75 0)
+		(fields_autoplaced yes)
 		(effects
 			(font
@@
 	(label "GPIO1"
 		(at 246.38 73.66 0)
+		(fields_autoplaced yes)
 		(effects
 			(font
@@
 	(label "V_RXD"
 		(at 322.58 139.7 0)
+		(fields_autoplaced yes)
 		(effects
 			(font
@@
 	(label "GPIO9"
 		(at 353.06 43.18 0)
+		(fields_autoplaced yes)
 		(effects
 			(font
@@
 	(label "DTR"
 		(at 195.58 68.58 0)
+		(fields_autoplaced yes)
 		(effects
 			(font
@@
 	(label "CHIP_PU"
 		(at 106.68 265.43 0)
+		(fields_autoplaced yes)
 		(effects
 			(font
@@
 			)
 		)
-		(property "Footprint" "23059082"
+		(property "Footprint" "2305908-2:23059082"
 			(at 41.91 332.41 0)
 			(effects
@@
 			)
 		)
-		(property "Footprint" "C17179450-2x3-IDC-Header:HDR-TH_6P-P2.54-V-F-R2-C3-S2.54-4"
+		(property "Footprint" "Connector_IDC:IDC-Header_2x03_P2.54mm_Vertical_SMD"
 			(at 257.81 81.28 0)
 			(effects
@@
 			)
 		)
-		(property "Footprint" "22139323"
+		(property "Footprint" "2213932-3:22139323"
 			(at 346.71 234.62 0)
 			(effects
